File: Hardware/Brightness_Meter/Brightness_Meter.kicad_sch (KiCad schematic)
At the start: 0 parts

Commit message: upload hardware
Other:
- added sheet adc (adc.kicad_sch)
- added sheet level shifting (level_shifting.kicad_sch)
- title: (none) -> ENTRY DIAGRAM
Changed lines of the file:
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@@
 (kicad_sch (version 20230121) (generator eeschema)
   (paper "A4")
-  (sheet (at 54.61 55.88) (size 26.67 13.97) (fields_autoplaced)
+  (title_block
+    (title "ENTRY DIAGRAM")
+    (date "2023-12-10")
+  )
+  (sheet (at 95.25 59.69) (size 26.67 13.97) (fields_autoplaced)
     (stroke (width 0.1524) (type solid))
     (fill (color 0 0 0 0.0000))
-    (property "Sheetname" "Power" (at 54.61 55.1684 0)
+    (property "Sheetname" "Power" (at 95.25 58.9784 0)
       (effects (font (size 1.27 1.27)) (justify left bottom))
     )
-    (property "Sheetfile" "power.kicad_sch" (at 54.61 70.4346 0)
+    (property "Sheetfile" "power.kicad_sch" (at 95.25 74.2446 0)
       (effects (font (size 1.27 1.27)) (justify left top))
     )
     (instances
-      (project "Measure_Lux"
+      (project "Brightness_Meter"
         (path "/f7cc1c24-a210-4fa3-a52b-f1d84e501e31" (page "2"))
       )
     )
   )
-  (sheet (at 99.06 55.88) (size 26.67 13.97) (fields_autoplaced)
+  (sheet (at 134.62 59.69) (size 26.67 66.04) (fields_autoplaced)
     (stroke (width 0.1524) (type solid))
     (fill (color 0 0 0 0.0000))
-    (property "Sheetname" "MCU" (at 99.06 55.1684 0)
+    (property "Sheetname" "MCU" (at 134.62 58.9784 0)
       (effects (font (size 1.27 1.27)) (justify left bottom))
     )
-    (property "Sheetfile" "mcu.kicad_sch" (at 99.06 70.4346 0)
+    (property "Sheetfile" "mcu.kicad_sch" (at 134.62 126.3146 0)
       (effects (font (size 1.27 1.27)) (justify left top))
     )
     (instances
-      (project "Measure_Lux"
+      (project "Brightness_Meter"
         (path "/f7cc1c24-a210-4fa3-a52b-f1d84e501e31" (page "3"))
       )
     )
   )
-  (sheet (at 139.7 55.88) (size 25.4 12.7) (fields_autoplaced)
+  (sheet (at 95.25 102.87) (size 26.67 15.24) (fields_autoplaced)
     (stroke (width 0.1524) (type solid))
     (fill (color 0 0 0 0.0000))
-    (property "Sheetname" "measure" (at 139.7 55.1684 0)
+    (property "Sheetname" "measure" (at 95.25 102.1584 0)
       (effects (font (size 1.27 1.27)) (justify left bottom))
     )
-    (property "Sheetfile" "measure.kicad_sch" (at 139.7 69.1646 0)
+    (property "Sheetfile" "measure.kicad_sch" (at 95.25 118.6946 0)
       (effects (font (size 1.27 1.27)) (justify left top))
     )
     (instances
-      (project "Measure_Lux"
+      (project "Brightness_Meter"
         (path "/f7cc1c24-a210-4fa3-a52b-f1d84e501e31" (page "4"))
       )
     )
   )
-  (sheet (at 180.34 57.15) (size 24.13 11.43) (fields_autoplaced)
+  (sheet (at 172.72 102.87) (size 26.67 15.24) (fields_autoplaced)
     (stroke (width 0.1524) (type solid))
     (fill (color 0 0 0 0.0000))
-    (property "Sheetname" "lcd" (at 180.34 56.4384 0)
+    (property "Sheetname" "level shifting" (at 172.72 102.1584 0)
       (effects (font (size 1.27 1.27)) (justify left bottom))
     )
-    (property "Sheetfile" "lcd.kicad_sch" (at 180.34 69.1646 0)
+    (property "Sheetfile" "level_shifting.kicad_sch" (at 172.72 118.6946 0)
       (effects (font (size 1.27 1.27)) (justify left top))
     )
     (instances
-      (project "Measure_Lux"
+      (project "Brightness_Meter"
+        (path "/f7cc1c24-a210-4fa3-a52b-f1d84e501e31" (page "8"))
+      )
+    )
+  )
+  (sheet (at 172.72 59.69) (size 26.67 13.97) (fields_autoplaced)
+    (stroke (width 0.1524) (type solid))
+    (fill (color 0 0 0 0.0000))
+    (property "Sheetname" "lcd" (at 172.72 58.9784 0)
+      (effects (font (size 1.27 1.27)) (justify left bottom))
+    )
+    (property "Sheetfile" "lcd.kicad_sch" (at 172.72 74.2446 0)
+      (effects (font (size 1.27 1.27)) (justify left top))
+    )
+    (instances
+      (project "Brightness_Meter"
+        (path "/f7cc1c24-a210-4fa3-a52b-f1d84e501e31" (page "6"))
+      )
+    )
+  )
+  (sheet (at 172.72 81.28) (size 26.67 15.24) (fields_autoplaced)
+    (stroke (width 0.1524) (type solid))
+    (fill (color 0 0 0 0.0000))
+    (property "Sheetname" "setting" (at 172.72 80.5684 0)
+      (effects (font (size 1.27 1.27)) (justify left bottom))
+    )
+    (property "Sheetfile" "setting.kicad_sch" (at 172.72 97.1046 0)
+      (effects (font (size 1.27 1.27)) (justify left top))
+    )
+    (instances
+      (project "Brightness_Meter"
+        (path "/f7cc1c24-a210-4fa3-a52b-f1d84e501e31" (page "7"))
+      )
+    )
+  )
+  (sheet (at 95.25 81.28) (size 26.67 13.97) (fields_autoplaced)
+    (stroke (width 0.1524) (type solid))
+    (fill (color 0 0 0 0.0000))
+    (property "Sheetname" "adc" (at 95.25 80.5684 0)
+      (effects (font (size 1.27 1.27)) (justify left bottom))
+    )
+    (property "Sheetfile" "adc.kicad_sch" (at 95.25 95.8346 0)
+      (effects (font (size 1.27 1.27)) (justify left top))
+    )
+    (instances
+      (project "Brightness_Meter"
         (path "/f7cc1c24-a210-4fa3-a52b-f1d84e501e31" (page "5"))
       )
     )
-  )
-  (sheet (at 214.63 57.15) (size 26.67 11.43) (fields_autoplaced)
-    (stroke (width 0.1524) (type solid))
-    (fill (color 0 0 0 0.0000))
-    (property "Sheetname" "setting" (at 214.63 56.4384 0)
-      (effects (font (size 1.27 1.27)) (justify left bottom))
-    )
-    (property "Sheetfile" "setting.kicad_sch" (at 214.63 69.1646 0)
-      (effects (font (size 1.27 1.27)) (justify left top))
-    )
-    (instances
-      (project "Measure_Lux"
-        (path "/f7cc1c24-a210-4fa3-a52b-f1d84e501e31" (page "6"))
-      )
-    )
