File: Hardware/Brightness_Meter/mcu.kicad_sch (KiCad schematic)
At the start: 5 parts, among them U1 STM32F030C8Tx

Commit message: upload hardware
Parts:
- added C16 (x3): 4.7uF/10V, Capacitor_SMD:C_0603_1608Metric_Pad1.08x0.95mm_HandSolder, symbol Device:C_Small
- added C16 (x4): 20pF/50V, Capacitor_SMD:C_0603_1608Metric_Pad1.08x0.95mm_HandSolder, symbol Device:C_Small
- added C16 (x5): 100nF/16V, Capacitor_SMD:C_0603_1608Metric_Pad1.08x0.95mm_HandSolder, symbol Device:C_Small
- added C16: 1uF/16V, Capacitor_SMD:C_0603_1608Metric_Pad1.08x0.95mm_HandSolder, symbol Device:C_Small
- added C16: 10nF/50V, Capacitor_SMD:C_0603_1608Metric_Pad1.08x0.95mm_HandSolder, symbol Device:C_Small
- added C16 (x2): 10uF/16V, Capacitor_SMD:C_0603_1608Metric_Pad1.08x0.95mm_HandSolder, symbol Device:C_Small
- added D3: Led_test, LED_SMD:LED_0805_2012Metric_Pad1.15x1.40mm_HandSolder, symbol Device:LED
- added D4: ZMM3V3, ZMM3V9_3V3:ZDO_ZMM_3p5x1p45_STM, symbol ZMM3V9_3V3:ZMM3V9
- added H1, H2, H3: MountingHole, MountingHole:MountingHole_3.2mm_M3_DIN965_Pad_TopBottom, symbol Mechanical:MountingHole
- added J2: Load Program, Connector_PinHeader_2.54mm:PinHeader_1x04_P2.54mm_Vertical, symbol Connector:Conn_01x04_Pin
- added R17: 1k/1%, Resistor_SMD:R_0603_1608Metric_Pad0.98x0.95mm_HandSolder, symbol Device:R_Small_US
- added Y1: 8MHz, Crystal:Crystal_SMD_EuroQuartz_MQ-4Pin_7.0x5.0mm, symbol Device:Crystal_GND24_Small
- added Y2: 32.768KHz, Crystal:Crystal_SMD_3215-2Pin_3.2x1.5mm, symbol Device:Crystal_Small
- R1, R2: value 0/0603/1% -> 0/1%; footprint Resistor_SMD:R_0201_0603Metric_Pad0.64x0.40mm_HandSolder -> Resistor_SMD:R_0603_1608Metric_Pad0.98x0.95mm_HandSolder
- R3: value 10k/0603/1% -> 10k/1%; footprint Resistor_SMD:R_0201_0603Metric_Pad0.64x0.40mm_HandSolder -> Resistor_SMD:R_0603_1608Metric_Pad0.98x0.95mm_HandSolder
- renumbered Reset to Reset1
Connections:
- net +3.3V: now also R3.1, U1.1 (VDD), U1.24 (VDD), U1.48 (VDD), U1.9 (VDDA), C16.1, C16.1, C16.1, C16.1, C16.1, C16.1, C16.1, C16.1, R17.1
- net GND: now also C16.1, C16.2, C16.2, C16.2, C16.2, C16.2, C16.2, C16.2, C16.2, C16.2, C16.2, C16.2, C16.2, C16.2, C16.2, C16.2, D4.2, J2.4 (Pin_4), Y1.2, Y1.4
- net RESET: now also C16.2
- net ADC_INO: now reaches U1.10 (PA0)
- net ADC_INO: now also C16.1, C16.1, D4.1
- net LED_INFO: now reaches U1.19 (PB1)
- net LED_TEST: now reaches U1.2 (PC13)
- net LED_TEST: now also D3.1 (K)
- net BUZZER: now reaches U1.20 (PB2)
- net SW_MODE: now reaches U1.21 (PB10)
- net SW_UP: now reaches U1.22 (PB11)
- net SW_SET: now reaches U1.25 (PB12)
- net SW_LEFT: now reaches U1.26 (PB13)
- net OSC32_IN: now reaches U1.3 (PC14)
- net OSC32_IN: now also C16.1, Y2.1
- net ADC_DATA: now reaches U1.30 (PA9)
- net ADC_CLK: now reaches U1.31 (PA10)
- net CHANGE_GAIN: now reaches U1.32 (PA11)
- net CHANGE_RESISTOR: now reaches U1.33 (PA12)
- net SWDIO: now reaches U1.34 (PA13)
- net SWDIO: now also J2.2 (Pin_2)
- net SWCLK: now reaches U1.37 (PA14)
- net SWCLK: now also J2.3 (Pin_3)
- net OSC32_OUT: now reaches U1.4 (PC15)
- net OSC32_OUT: now also C16.1, Y2.2
- net I2C_SCL: now reaches U1.42 (PB6)
- net I2C_SDA: now reaches U1.43 (PB7)
- net SW_RIGHT: now reaches U1.45 (PB8)
- net SW_DOWN: now reaches U1.46 (PB9)
- net OSC_IN: now reaches U1.5 (PF0)
- net OSC_IN: now also C16.1, Y1.1
- net OSC_OUT: now reaches U1.6 (PF1)
- net OSC_OUT: now also C16.1, Y1.3
- new net: D3.2 (A), R17.2
- new net +5V: C16.1, J2.1 (Pin_1)
- no-connect marks 0 -> 17
Other:
- note added: "FILTER"
- note added: "HOLE"
- note added: "LOAD PROGRAM"
- note added: "MCU"
- note added: "OSC"
- note added: "RESET - BOOT"
- title: (none) -> MCU
- moved on the sheet: R1, R2, R3, Reset1, U1
