File: Hardware/Brightness_Meter/measure.kicad_sch (KiCad schematic)
At the start: 0 parts

Commit message: upload hardware
Parts:
- added 5V: V_Ref, TestPoint:TestPoint_Pad_D1.5mm, symbol Connector:TestPoint
- added 5V: V_out, TestPoint:TestPoint_Pad_D1.5mm, symbol Connector:TestPoint
- added C14: 10pF/50V, Capacitor_SMD:C_0603_1608Metric_Pad1.08x0.95mm_HandSolder, symbol Device:C_Small
- added C14: 1uF/16V, Capacitor_SMD:C_0603_1608Metric_Pad1.08x0.95mm_HandSolder, symbol Device:C_Small
- added C16 (x4): 10uF/16V, Capacitor_SMD:C_0603_1608Metric_Pad1.08x0.95mm_HandSolder, symbol Device:C_Small
- added C16 (x4): 100nF/16V, Capacitor_SMD:C_0603_1608Metric_Pad1.08x0.95mm_HandSolder, symbol Device:C_Small
- added Q1 (x2): MMBT2222A, MMBT2222A:SOT23, symbol MMBT2222A:MMBT2222A
- added R1, R2: 0/1%, Resistor_SMD:R_0603_1608Metric_Pad0.98x0.95mm_HandSolder, symbol Device:R_US
- added R21: EVM-3ESX50B14, ul_EVM-3ESX50B14:EVM-3ESX50B14_PAN, symbol EVM-3ESX50B14:EVM-3ESX50B14
- added R22 (x2): 1k/1%, Resistor_SMD:R_0603_1608Metric_Pad0.98x0.95mm_HandSolder, symbol Device:R_Small_US
- added R22, R23, R28, R38: EVM-3E, ul_EVM-3ESX50B14:EVM-3ESX50B14_PAN, symbol EVM-3ESX50B14:EVM-3ESX50B14
- added R24: GL5528, OptoDevice:R_LDR_5.0x4.1mm_P3mm_Vertical, symbol Sensor_Optical:A9013
- added R4, R5, R6, R7, R8: R_Small_US, Resistor_SMD:R_0603_1608Metric_Pad0.98x0.95mm_HandSolder, symbol Device:R_Small_US
- added RG_1, RG_2: RG, TestPoint:TestPoint_Pad_D1.5mm, symbol Connector:TestPoint
- added RP_1, RP_2: RP, TestPoint:TestPoint_Pad_D1.5mm, symbol Connector:TestPoint
- added U3: MCP6002, MCP6002:SOIC127P599X173-8N, symbol MCP6002:MCP6002
- added U4: INA128, INA128UA:SOIC127P599X175-8N, symbol Amplifier_Instrumentation:INA128
Connections:
- new net: R6.1, R7.2, U3.3 (VINA+)
- new net: C14.1, R4.1, R5.2, U3.2 (VINA-)
- new net: C14.2, R5.1, R8.1, U3.1 (VOUTA)
- new net: Q1.1, R22.1 (x2)
- new net: Q1.3, R28.1
- new net: Q1.3, R38.1
- new net: R22.2, R38.2, RG_1.1, U4.1 (Rg)
- new net: R21.2, U3.5 (VINB+)
- new net: Q1.2, R22.1, RG_2.1, U4.8 (Rg)
- new net +5V: C16.1, C16.1, C16.1, C16.1, R21.3, R6.2, U3.8 (VDD), U4.7 (V+)
- new net -5V: C16.2, C16.2, C16.2, C16.2, U3.4 (VSS), U4.4 (V-)
- new net ADC_HX71OB: R1.2
- new net ADC_INO: R2.1
- new net CHANGE_GAIN: R22.2
- new net CHANGE_RESISTOR: R22.2
- new net CURRENT_SRC: C14.2, R23.2, R24.1, R28.2, R7.1, R8.2, RP_1.1, U4.3 (+)
- new net GND: C14.1, C16.1, C16.1, C16.1, C16.1, C16.2, C16.2, C16.2, C16.2, Q1.2, R21.1, R23.1, R24.2, R4.2, RP_2.1, U4.2 (-)
- new net VREF: 5V.1, U3.6 (VINB-), U3.7 (VOUTB), U4.5 (Ref)
- new net vout: 5V.1, R1.1, R2.2, U4.6
- no-connect marks 0 -> 4
Other:
- note added: "ADC"
- note added: "CURRENT SOURCE - VOLTAGE REFERENCE"
- note added: "DIFFERENCE AMPLIFIER"
- note added: "FILTER"
- note added: "TESTPOINT"
- title: (none) -> MEASURE
