File: Hardware/Brightness_Meter/power.kicad_sch (KiCad schematic)
At the start: 3 parts, among them U2 ICL7662CPA

Commit message: upload hardware
Parts:
- removed C1, C2: 10uF/16V, Capacitor_SMD:CP_Elec_4x5.4, symbol Device:C_Polarized_Small_US
- added -5V1: -5V, TestPoint:TestPoint_Pad_D1.5mm, symbol Connector:TestPoint
- added -5V2, 3.3V2, 5V2, Vin2: BLUE, LED_SMD:LED_0805_2012Metric_Pad1.15x1.40mm_HandSolder, symbol Device:LED
- added 3.3V1: 3.3V, TestPoint:TestPoint_Pad_D1.5mm, symbol Connector:TestPoint
- added 5V1: 5V, TestPoint:TestPoint_Pad_D1.5mm, symbol Connector:TestPoint
- added C1, C2, C6, C7: 10uF/16V, TAJA106K016RNJ:CAPMP3216X180N, symbol TAJA106K016RNJ:TAJA106K016RNJ
- added C10, C9: 4.7uF/25V, Capacitor_SMD:C_0603_1608Metric_Pad1.08x0.95mm_HandSolder, symbol Device:C_Small
- added C11, C12: 10nF/50V, Capacitor_SMD:C_0603_1608Metric_Pad1.08x0.95mm_HandSolder, symbol Device:C_Small
- added C13: 1nF/50V, Capacitor_SMD:C_0603_1608Metric_Pad1.08x0.95mm_HandSolder, symbol Device:C_Small
- added C14: 47pF/50V, Capacitor_SMD:C_0603_1608Metric_Pad1.08x0.95mm_HandSolder, symbol Device:C_Small
- added C15: 0.1uF/16V, Capacitor_SMD:C_0603_1608Metric_Pad1.08x0.95mm_HandSolder, symbol Device:C_Small
- added C16, C17: 47uF/6.3V, Capacitor_SMD:C_0603_1608Metric_Pad1.08x0.95mm_HandSolder, symbol Device:C_Small
- added C5, C8: 1uF/25V, TAJA105K025RNJ:CAPMP3216X180N, symbol TAJA105K025RNJ:TAJA105K025RNJ
- added C6: 22uF/25V, Capacitor_SMD:CP_Elec_6.3x5.4, symbol Device:C_Polarized_Small
- added D1, D2: SS34, SS34:DIOM4325X250N, symbol SS34:SS34
- added F1: Fuse_Small, Fuse:Fuse_1812_4532Metric_Pad1.30x3.40mm_HandSolder, symbol Device:Fuse_Small
- added GND1: GND, TestPoint:TestPoint_Pad_D1.5mm, symbol Connector:TestPoint
- added J1: JACK-DC, PRT-12748:SPARKFUN_PRT-12748, symbol PRT-12748:Jack_DC_5
- added L1: 6.8uH/2.2A, ul_SDE0604A-330M:IND_SDE0604A_5P8X5P2X4P5_BRN, symbol Inductor_5852:SDE0604A-330M
- added R11: 330k/1%, Resistor_SMD:R_0603_1608Metric_Pad0.98x0.95mm_HandSolder, symbol Device:R_Small_US
- added R12: 47k/1%, Resistor_SMD:R_0603_1608Metric_Pad0.98x0.95mm_HandSolder, symbol Device:R_Small_US
- added R13: 30k/1%, Resistor_SMD:R_0603_1608Metric_Pad0.98x0.95mm_HandSolder, symbol Device:R_Small_US
- added R14: 2.49k/1%, Resistor_SMD:R_0603_1608Metric_Pad0.98x0.95mm_HandSolder, symbol Device:R_Small_US
- added R15: 49.9k/1%, Resistor_SMD:R_0603_1608Metric_Pad0.98x0.95mm_HandSolder, symbol Device:R_Small_US
- added R16: 10k/1%, Resistor_SMD:R_0603_1608Metric_Pad0.98x0.95mm_HandSolder, symbol Device:R_Small_US
- added R17, R18: 1k/1%, Resistor_SMD:R_0603_1608Metric_Pad0.98x0.95mm_HandSolder, symbol Device:R_Small_US
- added R19, R27: 4.7k/1%, Resistor_SMD:R_0603_1608Metric_Pad0.98x0.95mm_HandSolder, symbol Device:R_Small_US
- added U6: LM1117DT-3.3, Package_TO_SOT_SMD:TO-252-3_TabPin2, symbol Regulator_Linear:LM1117DT-3.3
- added U7: TPS54331D, TPS54331D:SOIC127P599X175-8N, symbol TPS54331D:TPS54331D
- added Vin1: Vin, TestPoint:TestPoint_Pad_D1.5mm, symbol Connector:TestPoint
- U2: Availability Not in stock -> (none); Check_prices https://www.snapeda.com/parts/ICL7662CPA/Rochester+Electron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 -> (none); MF Rochester Electronics, LLC -> (none); MP ICL7662CPA -> (none); Package None -> (none); Price None -> (none); SnapEDA_Link https://www.snapeda.com/parts/ICL7662CPA/Rochester+Electron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 -> (none); URL (none) -> https://www.thegioiic.com/icl7662cba
Connections:
- net GND: now also 3.3V2.1 (K), 5V2.1 (K), C10.2, C11.2, C12.2, C14.2, C16.2, C17.2, C2.1, C5.2, C6.2, C6.2, C7.2, C8.2, C9.2, D1.A, D2.A, GND1.1, J1.2, J1.3, R12.2, R13.2, R16.2, R27.2, U6.1 (GND), U7.7 (GND), Vin2.1 (K)
- net at U2.2 (CAP+): now also C1.1
- net at U2.4 (CAP-): now also C1.2
- net +12V renamed +5V
- net +5V: now also 5V1.1, C16.1, C17.1, C5.1, C6.1, L1.1, R14.1, R17.1, U6.3 (VI)
- net -12V renamed -5V
- net -5V: now also -5V1.1, -5V2.1 (K), C2.2
- new net: R14.2, R15.1
- new net: R15.2, R16.1, U7.5 (VSENSE)
- new net: C15.1, D2.C, L1.2, U7.8 (PH)
- new net: C15.2, U7.1 (BOOT)
- new net: 5V2.2 (A), R17.2
- new net: R11.2, R12.1, U7.3 (EN)
- new net: C12.1, U7.4 (SS)
- new net: C13.1, C14.1, U7.6 (COMP)
- new net: C13.2, R13.1
- new net: R19.2, Vin2.2 (A)
- new net: F1.1, J1.1_1, J1.1_2
- new net: 3.3V2.2 (A), R18.2
- new net: -5V2.2 (A), R27.1
- new net +3.3V: 3.3V1.1, C7.1, C8.1, R18.1, U6.2 (VO)
- new net Vin: C10.1, C11.1, C6.1, C9.1, D1.C, F1.2, R11.1, R19.1, U7.2 (VIN), Vin1.1
Other:
- note added: "LDO"
- note added: "POWER LED"
- note added: "SWITCHING REGULATOR"
- note added: "TESTPOINT"
- note added: "VOLTAGE SUPPLY"
- title: (none) -> POWER
- moved on the sheet: U2
