File: Hardware/Brightness_Meter/setting.kicad_sch (KiCad schematic)
At the start: 0 parts

Commit message: upload hardware
Parts:
- added 3.3V: RED, LED_SMD:LED_0805_2012Metric_Pad1.15x1.40mm_HandSolder, symbol Device:LED
- added BZ1: Buzzer, Buzzer_Beeper:Buzzer_12x9.5RM7.6, symbol Device:Buzzer
- added C16 (x6): 100nF/16V, Capacitor_SMD:C_0603_1608Metric_Pad1.08x0.95mm_HandSolder, symbol Device:C_Small
- added D1: SS34, SS34:DIOM4325X250N, symbol SS34:SS34
- added DOWN1: DOWN, TL3300CF260Q:SW_TL3300CF260Q, symbol TL3300CF260Q:SW_SMD_12_12
- added LEFT1: LEFT, TL3300CF260Q:SW_TL3300CF260Q, symbol TL3300CF260Q:SW_SMD_12_12
- added MODE1: MODE, TL3300CF260Q:SW_TL3300CF260Q, symbol TL3300CF260Q:SW_SMD_12_12
- added Q1: MMBT2222A, MMBT2222A:SOT23, symbol MMBT2222A:MMBT2222A
- added R18 (x2): 1k/1%, Resistor_SMD:R_0603_1608Metric_Pad0.98x0.95mm_HandSolder, symbol Device:R_Small_US
- added R3 (x6): 10k/1%, Resistor_SMD:R_0603_1608Metric_Pad0.98x0.95mm_HandSolder, symbol Device:R_US
- added RIGHT1: RIGHT, TL3300CF260Q:SW_TL3300CF260Q, symbol TL3300CF260Q:SW_SMD_12_12
- added SET1: SET, TL3300CF260Q:SW_TL3300CF260Q, symbol TL3300CF260Q:SW_SMD_12_12
- added UP1: UP, TL3300CF260Q:SW_TL3300CF260Q, symbol TL3300CF260Q:SW_SMD_12_12
Connections:
- new net: 3.3V.1 (K), R18.1
- new net: Q1.1, R18.2
- new net: BZ1.2 (+), D1.A, Q1.3
- new net +3.3V: R3.2, R3.2, R3.2, R3.2, R3.2, R3.2
- new net +5V: BZ1.1 (-), D1.C
- new net BUZZER: R18.1
- new net GND: 3.3V.2 (A), C16.1, C16.1, C16.1, C16.1, C16.1, C16.1, DOWN1.1, DOWN1.2, LEFT1.1, LEFT1.2, MODE1.1, MODE1.2, Q1.2, RIGHT1.1, RIGHT1.2, SET1.1, SET1.2, UP1.1, UP1.2
- new net LED_INFO: R18.2
- new net SW_DOWN: C16.2, DOWN1.3, DOWN1.4, R3.1
- new net SW_LEFT: C16.2, LEFT1.3, LEFT1.4, R3.1
- new net SW_MODE: C16.2, MODE1.3, MODE1.4, R3.1
- new net SW_RIGHT: C16.2, R3.1, RIGHT1.3, RIGHT1.4
- new net SW_SET: C16.2, R3.1, SET1.3, SET1.4
- new net SW_UP: C16.2, R3.1, UP1.3, UP1.4
Other:
- note added: "SWITCH"
- note added: "WARNNING"
- title: (none) -> SETTING
